File: LPC800_TSSOP_breadboard_mini.brd (EAGLE design)
At the start: 26 x 15.9 mm, 16 parts, among them Q1 12MHz

Commit message: * fixed some small mistakes
Parts:
- added LOGO1: OSHW_LOGO_FILLX0150-NT, ohw-logo:OSHW_FILLX150_NOTEXT
Other:
- board text added: "14"
- board text added: "V2015.11.22"
- board text removed: "V2014.10.09"
Changed lines of the file:
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@@
 <?xml version="1.0" encoding="utf-8"?>
 <!DOCTYPE eagle SYSTEM "eagle.dtd">
-<eagle version="7.1.0">
+<eagle version="7.3.0">
 <drawing>
 <settings>
@@
 <wire x1="0" y1="15.875" x2="0" y2="0" width="0" layer="20"/>
 <wire x1="0" y1="0" x2="26.035" y2="0" width="0" layer="20"/>
-<text x="23.1775" y="3.4925" size="1.016" layer="22" rot="MR0">V2014.10.09</text>
+<text x="23.1775" y="3.4925" size="1.016" layer="22" font="vector" rot="MR0">V2015.11.22</text>
 <text x="1.905" y="3.175" size="0.6096" layer="25" rot="R90">17</text>
 <text x="4.445" y="3.175" size="0.6096" layer="25" rot="R90">13</text>
 <text x="6.985" y="3.175" size="0.6096" layer="25" rot="R90">12</text>
 <text x="9.525" y="3.175" size="0.6096" layer="25" rot="R90">5</text>
-<text x="13.0175" y="3.175" size="0.6096" layer="25" rot="R90">4</text>
-<text x="15.5575" y="3.175" size="0.6096" layer="25" rot="R90">3</text>
+<text x="12.065" y="3.175" size="0.6096" layer="25" rot="R90">4</text>
+<text x="14.605" y="3.175" size="0.6096" layer="25" rot="R90">3</text>
 <text x="17.145" y="3.175" size="0.6096" layer="25" rot="R90">2</text>
 <text x="19.685" y="3.175" size="0.6096" layer="25" rot="R90">11</text>
@@
 <text x="21.59" y="12.7" size="0.6096" layer="25" rot="R270">1</text>
 <text x="19.05" y="12.7" size="0.6096" layer="25" rot="R270">9</text>
-<text x="17.4625" y="12.7" size="0.6096" layer="25" rot="R270">8</text>
+<text x="16.51" y="12.7" size="0.6096" layer="25" rot="R270">8</text>
 <text x="8.89" y="12.7" size="0.6096" layer="25" rot="R270">7</text>
 <text x="6.35" y="12.7" size="0.6096" layer="25" rot="R270">6</text>
 <text x="3.81" y="12.7" size="0.6096" layer="25" rot="R270">0</text>
-<text x="1.27" y="12.7" size="0.6096" layer="25" rot="R270">15</text>
+<text x="1.27" y="12.7" size="0.6096" layer="25" rot="R270">14</text>
 <text x="11.43" y="12.7" size="0.6096" layer="25" rot="R270">V-</text>
 <text x="13.97" y="12.7" size="0.6096" layer="25" rot="R270">V+</text>
@@
 <element name="U$3" library="SquantorButtons" package="TD-85XU" value="TACT_2PIN" x="4.1275" y="9.8425" smashed="yes" rot="R180"/>
 <element name="U$4" library="SquantorButtons" package="TD-85XU" value="TACT_2PIN" x="4.1275" y="6.0325" smashed="yes" rot="R180"/>
+<element name="LOGO1" library="ohw-logo" package="OSHW_FILLX150_NOTEXT" value="OSHW_LOGO_FILLX0150-NT" x="14.1605" y="3.9116" rot="MR0"/>
 </elements>
 <signals>
