File: kicad/LPC82X_JHI33_2layer/LPC82X_JHI33_2layer.kicad_pcb (KiCad board)
At the start: 2 copper layers, 23.6 x 23.5 mm, 24 parts, among them J1 Conn_02x09_Odd_Even, J2 Conn_02x09_Odd_Even, J3 JTAG_2X05, U1 LPC824M201JHI33, Y1 12MHz

Commit message: updated version number
Parts:
- N2: value 20181029 -> 20181102
Changed lines of the file:
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@@
       (effects (font (size 1 1) (thickness 0.15)) (justify mirror))
     )
-    (fp_text value 20181029 (at -0.4 0.137362 270) (layer B.SilkS)
+    (fp_text value 20181102 (at -0.4 0.137362 270) (layer B.SilkS)
       (effects (font (size 1 1) (thickness 0.15)) (justify mirror))
     )
