File: hardware/LPC82X_JDH20/LPC82X_JDH20.kicad_pcb (KiCad board)
At the start: 2 copper layers, 18.7 x 23.8 mm, 24 parts, among them J1 Conn_01x09, J2 JTAG_2X05, J3 Conn_01x09, U1 LPC824M201JDH20, Y1 12MHz

Commit message: added named connectors for LPC82XJDH20 breakout
Parts:
- J1: footprint SquantorConnectors:Header-0254-1X09-H010 -> SquantorConnectorsNamed:LPC82XJDH20_breakout_left; moved to B.Cu
- J2: value JTAG_2X05 -> JTAG_2X05_IN
- J3: footprint SquantorConnectors:Header-0254-1X09-H010 -> SquantorConnectorsNamed:LPC82XJDH20_breakout_right; moved to B.Cu
- N2: value 20190121 -> 20190410
Connections:
- net VDD renamed /VDD
- net VSS renamed /VSS
Routing:
- added copper zone on F.Cu, net /VDD
- removed copper zone on F.Cu, net /VSS
