File: hardware/LPC82X_JDH20/LPC82X_JDH20.kicad_pcb (KiCad board)
At the start: 2 copper layers, 18.7 x 23.8 mm, 24 parts, among them J1 Conn_01x09, J2 JTAG_2X05_IN, J3 Conn_01x09, U1 LPC824M201JDH20, Y1 12MHz

Commit message: updated versionnumber
Parts:
- N2: value 20190410 -> 20190411
Changed lines of the file:
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@@
       (effects (font (size 1 1) (thickness 0.15)) (justify mirror))
     )
-    (fp_text value 20190410 (at -0.4 0.1) (layer B.SilkS)
+    (fp_text value 20190411 (at -0.4 0.1) (layer B.SilkS)
       (effects (font (size 1 1) (thickness 0.15)) (justify mirror))
     )
