File: hardware/LPC82X_JDH20/LPC82X_JDH20.sch (KiCad schematic (older format))
At the start: 24 parts, among them J1 Conn_01x09, J2 JTAG_2X05, J3 Conn_01x09, U1 LPC824M201JDH20, Y1 12MHz

Commit message: added named connectors for LPC82XJDH20 breakout
Parts:
- removed J2: JTAG_2X05, SquantorConnectors:Header-0127-2X05-H006, symbol SquantorConnectors:JTAG_2X05
- added J2: JTAG_2X05_IN, SquantorConnectors:Header-0127-2X05-H006, symbol SquantorConnectors:JTAG_2X05_IN
- J1: footprint SquantorConnectors:Header-0254-1X09-H010 -> SquantorConnectorsNamed:LPC82XJDH20_breakout_left; symbol Connector_Generic:Conn_01x09 -> SquantorConnectorsNamed:LPC82XJDH20_breakout_left
- J3: footprint SquantorConnectors:Header-0254-1X09-H010 -> SquantorConnectorsNamed:LPC82XJDH20_breakout_right; symbol Connector_Generic:Conn_01x09 -> SquantorConnectorsNamed:LPC82XJDH20_breakout_right
- N2: value 20190121 -> 20190410
Connections:
- net VDD: now also J2.1 (VCC)
- net VSS: now also J2.3 (GND), J2.5 (GND), J2.9 (GNDDET)
- net at R6.1: now also J2.10 (nRESET)
- net at R4.1: now also J2.2 (SWDIO/TMS)
- net at R5.1: now also J2.4 (SWDCLK/TCK)
- no-connect marks 0 -> 2
Other:
- moved on the sheet: J1, J3

Commit message: updated versionnumber
Parts:
- N2: value 20190410 -> 20190411
Changed lines of the file:
@@
 P 850 7700
 F 0 "N2" H 850 7800 60  0000 C CNN
-F 1 "20190410" H 850 7700 60  0000 C CNN
+F 1 "20190411" H 850 7700 60  0000 C CNN
 F 2 "SquantorLabels:Label_version" H 850 7700 60  0001 C CNN
 F 3 "" H 850 7700 60  0001 C CNN
