File: hardware/LPC82X_JHI33/LPC82X_JHI33.kicad_pcb (KiCad board)
At the start: 2 copper layers, 23.6 x 23.5 mm, 24 parts, among them J1 LPC82XJHI33_LEFT, J2 LPC82XJHI33_RIGHT, J3 JTAG_2X05, U1 LPC824M201JHI33, Y1 12MHz

Commit message: updated versionnumber
Parts:
- N2: value 20190411 -> 20190514
Changed lines of the file:
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@@
     (add_net "Net-(J3-Pad2)")
     (add_net "Net-(J3-Pad4)")
+    (add_net "Net-(J3-Pad6)")
+    (add_net "Net-(J3-Pad7)")
+    (add_net "Net-(J3-Pad8)")
   )
   (module SquantorConnectorsNamed:LPC82XJHI33_breakout_right (layer F.Cu)
@@
       (effects (font (size 1 1) (thickness 0.15)) (justify mirror))
     )
-    (fp_text value 20190411 (at -0.4 0.137362 180) (layer B.SilkS)
+    (fp_text value 20190514 (at -0.4 0.137362 180) (layer B.SilkS)
       (effects (font (size 1 1) (thickness 0.15)) (justify mirror))
     )
